File: PCB/v1.0/MDAS_Controller_V1.brd (EAGLE design)
At the start: 54.8 x 55.9 mm, 32 parts, among them IC1 7805TV, U1 TPS70912QDBVRQ1, U2 TPS70912QDBVRQ1, U3 OPA2333-Q1_D_8, U4 OPA2333-Q1_D_8

Commit message: PCB changes
Parts:
- added C7: .1uF, adafruit:C0603
- added CAN_TRANSCIEVER1: TCAN332, Texas Instruments_By_element14_Batch_1:SOIC127P600X172-8N
- added R14: 120, adafruit:0207/10
- added SV2: (no value), con-lstb:MA06-1
Connections:
- net CANH renamed CAN0H
- net CANL renamed CAN0L
- net RX renamed RX0
- net TX renamed TX0
- new net CAN1H: CAN_TRANSCIEVER1.7, DB9.8, R14.1
- new net CAN1L: CAN_TRANSCIEVER1.6, DB9.1, R14.2
- new net RX1: CAN_TRANSCIEVER1.4, SV2.6
- new net TX1: CAN_TRANSCIEVER1.1, SV2.5
- net 3V3: now also C7.1, CAN_TRANSCIEVER1.3
- net GND: now also C7.2, CAN_TRANSCIEVER1.2
Routing:
- net CAN0H: track 19.5 -> 14.0 mm
Changed lines of the file:
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@@
 <?xml version="1.0" encoding="utf-8"?>
 <!DOCTYPE eagle SYSTEM "eagle.dtd">
-<eagle version="9.0.0">
+<eagle version="9.1.0">
 <drawing>
 <settings>
@@
 <param name="checkStop" value="0"/>
 <param name="checkValues" value="0"/>
+<param name="checkNames" value="1"/>
+<param name="checkWireStubs" value="1"/>
+<param name="checkPolygonWidth" value="0"/>
 <param name="useDiameter" value="13"/>
 <param name="maxErrors" value="50"/>
@@
 <param name="tpViaShape" value="round"/>
 <param name="PrefDir.1" value="a"/>
-<param name="PrefDir.2" value="a"/>
+<param name="PrefDir.2" value="0"/>
 <param name="PrefDir.3" value="0"/>
 <param name="PrefDir.4" value="0"/>
@@
 <param name="PrefDir.13" value="0"/>
 <param name="PrefDir.14" value="0"/>
-<param name="PrefDir.15" value="-"/>
+<param name="PrefDir.15" value="0"/>
 <param name="PrefDir.16" value="-"/>
 <param name="cfVia" value="8"/>
@@
 <element name="INPUTS" library="SparkFun-Connectors" package="1X06-1MM" value="" x="34.29" y="3.81"/>
 <element name="D1" library="diode" library_urn="urn:adsk.eagle:library:210" package="DO41-10" package3d_urn="urn:adsk.eagle:package:43336/1" value="1N4004" x="22.86" y="34.925" rot="R180"/>
+<element name="CAN_TRANSCIEVER1" library="Texas Instruments_By_element14_Batch_1" package="SOIC127P600X172-8N" value="TCAN332" x="3.8735" y="-7.8105"/>
+<element name="R14" library="adafruit" library_urn="urn:adsk.eagle:library:420" package="0207/10" value="120" x="10.414" y="-17.5895"/>
+<element name="C7" library="adafruit" library_urn="urn:adsk.eagle:library:420" package="C0603" value=".1uF" x="1.2065" y="-16.8275"/>
+<element name="SV2" library="con-lstb" library_urn="urn:adsk.eagle:library:162" package="MA06-1" package3d_urn="urn:adsk.eagle:package:8340/1" value="" x="7.874" y="-29.7815">
+<attribute name="MF" value="" x="7.874" y="-29.7815" size="1.778" layer="27" display="off"/>
+<attribute name="MPN" value="" x="7.874" y="-29.7815" size="1.778" layer="27" display="off"/>
+<attribute name="OC_FARNELL" value="unknown" x="7.874" y="-29.7815" size="1.778" layer="27" display="off"/>
+<attribute name="OC_NEWARK" value="unknown" x="7.874" y="-29.7815" size="1.778" layer="27" display="off"/>
+</element>
 </elements>
 <signals>
@@
 <via x="12.065" y="24.765" extent="1-16" drill="0.35"/>
 <contactref element="D1" pad="A"/>
+<contactref element="CAN_TRANSCIEVER1" pad="2"/>
+<contactref element="C7" pad="2"/>
+<wire x1="17.78" y1="34.925" x2="27.94" y2="44.3" width="0" layer="19" extent="1-1"/>
+<wire x1="19.05" y1="31.75" x2="17.78" y2="34.925" width="0" layer="19" extent="1-1"/>
+<wire x1="21.59" y1="21.995" x2="20.535" y2="31.115" width="0" layer="19" extent="1-1"/>
+<wire x1="20.32" y1="11.3999" x2="21.59" y2="19.915" width="0" layer="19" extent="1-1"/>
+<wire x1="19.51" y1="5.08" x2="20.74" y2="8.89" width="0" layer="19" extent="1-1"/>
+<wire x1="15.875" y1="8.89" x2="20.32" y2="10.16" width="0" layer="19" extent="1-1"/>
+<wire x1="12.7" y1="17.36" x2="15.24" y2="11.3999" width="0" layer="19" extent="1-1"/>
+<wire x1="12.065" y1="24.765" x2="12.7" y2="18.415" width="0" layer="19" extent="1-1"/>
+<wire x1="36.09" y1="21.59" x2="26.035" y2="20.955" width="0" layer="19" extent="1-1"/>
+<wire x1="36.09" y1="26.035" x2="36.09" y2="21.59" width="0" layer="19" extent="1-1"/>
+<wire x1="44.665" y1="19.05" x2="37.465" y2="21.59" width="0" layer="19" extent="1-1"/>
+<wire x1="39.8158" y1="5.715" x2="39.4462" y2="8.89" width="0" layer="19" extent="1-15"/>
+<wire x1="1.4097" y1="-7.1755" x2="19.51" y2="3.35" width="0" layer="19" extent="1-1"/>
+<wire x1="2.0565" y1="-16.8275" x2="1.4097" y2="-7.1755" width="0" layer="19" extent="1-1"/>
 </signal>
-<signal name="CANL">
+<signal name="CAN0L">
 <contactref element="CAN_TRANSCIEVER" pad="6"/>
 <contactref element="R1" pad="2"/>
@@
 <wire x1="26.035" y1="32.385" x2="26.035" y2="30.48" width="0.508" layer="1"/>
 </signal>
-<signal name="CANH">
-<contactref element="CAN_TRANSCIEVER" pad="7"/>
-<contactref element="R1" pad="1"/>
-<contactref element="DB9" pad="7"/>
-<wire x1="26.56" y1="47.14" x2="26.56" y2="42.02" width="0.508" layer="1"/>
-<wire x1="26.56" y1="42.02" x2="30.48" y2="38.1" width="0.508" layer="1"/>
-<wire x1="30.48" y1="38.1" x2="30.48" y2="32.385" width="0.508" layer="1"/>
-<wire x1="30.48" y1="32.385" x2="29.21" y2="31.115" width="0.508" layer="1"/>
-<wire x1="29.21" y1="31.115" x2="27.8638" y2="31.115" width="0.508" layer="1"/>
-</signal>
 <signal name="12V">
 <contactref element="DB9" pad="9"/>
@@
 <via x="11.43" y="26.67" extent="1-16" drill="0.35"/>
 </signal>
-<signal name="RX">
+<signal name="RX0">
 <contactref element="A1" pad="5"/>
 <contactref element="CAN_TRANSCIEVER" pad="4"/>
@@
 <wire x1="4.445" y1="16.51" x2="5.715" y2="17.78" width="0.254" layer="1"/>
 </signal>
-<signal name="TX">
+<signal name="TX0">
 <contactref element="A1" pad="6"/>
 <contactref element="CAN_TRANSCIEVER" pad="1"/>
@@
 <wire x1="22.9362" y1="29.845" x2="19.05" y2="29.845" width="0.508" layer="1"/>
 <wire x1="44.3738" y1="12.7" x2="43.815" y2="12.7" width="0.254" layer="1"/>
+<contactref element="CAN_TRANSCIEVER1" pad="3"/>
+<contactref element="C7" pad="1"/>
+<wire x1="32.385" y1="15.7988" x2="43.815" y2="12.7" width="0" layer="19" extent="1-1"/>
+<wire x1="22.9362" y1="29.845" x2="32.385" y2="17.78" width="0" layer="19" extent="1-1"/>
+<wire x1="4.445" y1="26.67" x2="19.05" y2="29.845" width="0" layer="19" extent="1-1"/>
+<wire x1="1.4097" y1="-8.4455" x2="4.445" y2="26.67" width="0" layer="19" extent="1-1"/>
+<wire x1="0.3565" y1="-16.8275" x2="1.4097" y2="-8.4455" width="0" layer="19" extent="1-1"/>
 </signal>
 <signal name="SCL">
@@
 <wire x1="44.3738" y1="3.9488" x2="44.3738" y2="8.89" width="0.4064" layer="1"/>
 </signal>
+<signal name="CAN0H">
+<contactref element="CAN_TRANSCIEVER" pad="7"/>
+<contactref element="R1" pad="1"/>
+<wire x1="30.48" y1="38.1" x2="30.48" y2="32.385" width="0.508" layer="1"/>
+<wire x1="30.48" y1="32.385" x2="29.21" y2="31.115" width="0.508" layer="1"/>
+<wire x1="29.21" y1="31.115" x2="27.8638" y2="31.115" width="0.508" layer="1"/>
+<contactref element="DB9" pad="7"/>
+<wire x1="26.56" y1="47.14" x2="26.56" y2="42.02" width="0.508" layer="1"/>
+<wire x1="30.48" y1="38.1" x2="26.56" y2="42.02" width="0" layer="19" extent="1-1"/>
+</signal>
+<signal name="CAN1H">
+<contactref element="CAN_TRANSCIEVER1" pad="7"/>
+<contactref element="R14" pad="1"/>
+<contactref element="DB9" pad="8"/>
+<wire x1="6.3373" y1="-7.1755" x2="29.32" y2="47.14" width="0" layer="19" extent="1-1"/>
+<wire x1="5.334" y1="-17.5895" x2="6.3373" y2="-7.1755" width="0" layer="19" extent="1-1"/>
+</signal>
+<signal name="CAN1L">
+<contactref element="CAN_TRANSCIEVER1" pad="6"/>
+<contactref element="R14" pad="2"/>
+<contactref element="DB9" pad="1"/>
+<wire x1="6.3373" y1="-8.4455" x2="22.4" y2="44.3" width="0" layer="19" extent="1-1"/>
+<wire x1="15.494" y1="-17.5895" x2="6.3373" y2="-8.4455" width="0" layer="19" extent="1-1"/>
+</signal>
+<signal name="RX1">
+<contactref element="SV2" pad="6"/>
+<contactref element="CAN_TRANSCIEVER1" pad="4"/>
+<wire x1="1.4097" y1="-9.7155" x2="14.224" y2="-29.7815" width="0" layer="19" extent="1-1"/>
+</signal>
+<signal name="TX1">
+<contactref element="SV2" pad="5"/>
+<contactref element="CAN_TRANSCIEVER1" pad="1"/>
+<wire x1="1.4097" y1="-5.9055" x2="11.684" y2="-29.7815" width="0" layer="19" extent="1-1"/>
+</signal>
 </signals>
+<mfgpreviewcolors>
+<mfgpreviewcolor name="soldermaskcolor" color="0xC8008000"/>
+<mfgpreviewcolor name="silkscreencolor" color="0xFFFEFEFE"/>
+<mfgpreviewcolor name="backgroundcolor" color="0xFF282828"/>
+<mfgpreviewcolor name="coppercolor" color="0xFFFFBF00"/>
+<mfgpreviewcolor name="substratecolor" color="0xFF786E46"/>
+</mfgpreviewcolors>
 <errors>
 </errors>
