File: PCB/v1.0/MDAS_Controller_V1.sch (EAGLE design)
At the start: 32 parts, among them IC1 7805TV, U1 TPS70912QDBVRQ1, U2 TPS70912QDBVRQ1, U3 OPA2333-Q1_D_8, U4 OPA2333-Q1_D_8

Commit message: PCB changes
Parts:
- added C7: .1uF, adafruit:C-USC0603
- added CAN_TRANSCIEVER1: TCAN332, Texas Instruments_By_element14_Batch_1:TCAN332
- added R14: 120, adafruit:R-US_0207/10
- added SV2: (no value), con-lstb:MA06-1
Connections:
- net CANH renamed CAN0H
- net CANL renamed CAN0L
- net RX renamed RX0
- net TX renamed TX0
- new net CAN1H: CAN_TRANSCIEVER1.CANH, DB9.8, R14.1
- new net CAN1L: CAN_TRANSCIEVER1.CANL, DB9.1, R14.2
- new net RX1: CAN_TRANSCIEVER1.RXD, SV2.6
- new net TX1: CAN_TRANSCIEVER1.TXD, SV2.5
- net 3V3: now also C7.1, CAN_TRANSCIEVER1.VCC
- net GND: now also C7.2, CAN_TRANSCIEVER1.GND
Changed lines of the file:
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@@
 <?xml version="1.0" encoding="utf-8"?>
 <!DOCTYPE eagle SYSTEM "eagle.dtd">
-<eagle version="9.0.0">
+<eagle version="9.1.0">
 <drawing>
 <settings>
@@
 <part name="INPUTS" library="SparkFun-Connectors" deviceset="M06" device="SMD-1MM"/>
 <part name="D1" library="diode" library_urn="urn:adsk.eagle:library:210" deviceset="1N4004" device="" package3d_urn="urn:adsk.eagle:package:43336/1"/>
+<part name="CAN_TRANSCIEVER1" library="Texas Instruments_By_element14_Batch_1" deviceset="TCAN332" device=""/>
+<part name="R14" library="adafruit" library_urn="urn:adsk.eagle:library:420" deviceset="R-US_" device="0207/10" value="120"/>
+<part name="C7" library="adafruit" library_urn="urn:adsk.eagle:library:420" deviceset="C-US" device="C0603" value=".1uF"/>
+<part name="SV2" library="con-lstb" library_urn="urn:adsk.eagle:library:162" deviceset="MA06-1" device="" package3d_urn="urn:adsk.eagle:package:8340/1"/>
 </parts>
 <sheets>
@@
 <instance part="INPUTS" gate="G$1" x="99.06" y="48.26" rot="R180"/>
 <instance part="D1" gate="1" x="7.62" y="99.06"/>
+<instance part="CAN_TRANSCIEVER1" gate="G$1" x="-5.08" y="134.62"/>
+<instance part="R14" gate="G$1" x="27.94" y="132.08" rot="R270"/>
+<instance part="C7" gate="G$1" x="-22.86" y="129.54" rot="R180"/>
+<instance part="SV2" gate="1" x="-30.48" y="5.08" rot="R270"/>
 </instances>
 <busses>
@@
 <label x="137.16" y="109.22" size="1.778" layer="95"/>
 </segment>
-</net>
-<net name="CANL" class="0">
+<segment>
+<pinref part="CAN_TRANSCIEVER1" gate="G$1" pin="GND"/>
+<wire x1="-20.32" y1="134.62" x2="-22.86" y2="134.62" width="0.1524" layer="91"/>
+<wire x1="-22.86" y1="134.62" x2="-25.4" y2="134.62" width="0.1524" layer="91"/>
+<wire x1="-25.4" y1="134.62" x2="-25.4" y2="116.84" width="0.1524" layer="91"/>
+<wire x1="-25.4" y1="116.84" x2="-43.18" y2="116.84" width="0.1524" layer="91"/>
+<label x="-25.4" y="134.62" size="1.778" layer="95"/>
+<pinref part="C7" gate="G$1" pin="2"/>
+<junction x="-22.86" y="134.62"/>
+</segment>
+</net>
+<net name="CAN0L" class="0">
 <segment>
 <pinref part="CAN_TRANSCIEVER" gate="G$1" pin="CANL"/>
@@
 <wire x1="-10.16" y1="78.74" x2="0" y2="78.74" width="0.1524" layer="91"/>
 <label x="-7.62" y="78.74" size="1.778" layer="95"/>
-</segment>
-</net>
-<net name="CANH" class="0">
-<segment>
-<pinref part="CAN_TRANSCIEVER" gate="G$1" pin="CANH"/>
-<wire x1="63.5" y1="83.82" x2="73.66" y2="83.82" width="0.1524" layer="91"/>
-<wire x1="73.66" y1="83.82" x2="73.66" y2="86.36" width="0.1524" layer="91"/>
-<label x="66.04" y="83.82" size="1.778" layer="95"/>
-<pinref part="R1" gate="G$1" pin="1"/>
-<wire x1="78.74" y1="86.36" x2="73.66" y2="86.36" width="0.1524" layer="91"/>
-</segment>
-<segment>
-<pinref part="DB9" gate="G$1" pin="7"/>
-<wire x1="15.24" y1="76.2" x2="20.32" y2="76.2" width="0.1524" layer="91"/>
-<label x="15.24" y="76.2" size="1.778" layer="95"/>
 </segment>
 </net>
@@
 </segment>
 </net>
-<net name="RX" class="0">
+<net name="RX0" class="0">
 <segment>
 <pinref part="A1" gate="G$1" pin="P$5"/>
@@
 </segment>
 </net>
-<net name="TX" class="0">
+<net name="TX0" class="0">
 <segment>
 <pinref part="A1" gate="G$1" pin="P$6"/>
@@
 <label x="198.12" y="147.32" size="1.778" layer="95"/>
 </segment>
+<segment>
+<pinref part="CAN_TRANSCIEVER1" gate="G$1" pin="VCC"/>
+<wire x1="-20.32" y1="127" x2="-22.86" y2="127" width="0.1524" layer="91"/>
+<wire x1="-22.86" y1="127" x2="-22.86" y2="114.3" width="0.1524" layer="91"/>
+<wire x1="-22.86" y1="114.3" x2="-40.64" y2="114.3" width="0.1524" layer="91"/>
+<label x="-22.86" y="127" size="1.778" layer="95"/>
+<pinref part="C7" gate="G$1" pin="1"/>
+<junction x="-22.86" y="127"/>
+</segment>
 </net>
 <net name="SCL" class="0">
@@
 </segment>
 </net>
+<net name="CAN0H" class="0">
+<segment>
+<pinref part="CAN_TRANSCIEVER" gate="G$1" pin="CANH"/>
+<wire x1="63.5" y1="83.82" x2="73.66" y2="83.82" width="0.1524" layer="91"/>
+<wire x1="73.66" y1="83.82" x2="73.66" y2="86.36" width="0.1524" layer="91"/>
+<label x="66.04" y="83.82" size="1.778" layer="95"/>
+<pinref part="R1" gate="G$1" pin="1"/>
+<wire x1="78.74" y1="86.36" x2="73.66" y2="86.36" width="0.1524" layer="91"/>
+</segment>
+<segment>
+<pinref part="DB9" gate="G$1" pin="7"/>
+<wire x1="15.24" y1="76.2" x2="20.32" y2="76.2" width="0.1524" layer="91"/>
+<label x="15.24" y="76.2" size="1.778" layer="95"/>
+</segment>
+</net>
+<net name="CAN1H" class="0">
+<segment>
+<pinref part="CAN_TRANSCIEVER1" gate="G$1" pin="CANH"/>
+<wire x1="12.7" y1="134.62" x2="22.86" y2="134.62" width="0.1524" layer="91"/>
+<wire x1="22.86" y1="134.62" x2="22.86" y2="137.16" width="0.1524" layer="91"/>
+<label x="15.24" y="134.62" size="1.778" layer="95"/>
+<pinref part="R14" gate="G$1" pin="1"/>
+<wire x1="27.94" y1="137.16" x2="22.86" y2="137.16" width="0.1524" layer="91"/>
+</segment>
+<segment>
+<pinref part="DB9" gate="G$1" pin="8"/>
+<wire x1="15.24" y1="73.66" x2="20.32" y2="73.66" width="0.1524" layer="91"/>
+<wire x1="20.32" y1="73.66" x2="20.32" y2="109.22" width="0.1524" layer="91"/>
+<wire x1="20.32" y1="109.22" x2="27.94" y2="109.22" width="0.1524" layer="91"/>
+<label x="27.94" y="109.22" size="1.778" layer="95"/>
+</segment>
+</net>
+<net name="CAN1L" class="0">
+<segment>
+<pinref part="CAN_TRANSCIEVER1" gate="G$1" pin="CANL"/>
+<wire x1="12.7" y1="127" x2="27.94" y2="127" width="0.1524" layer="91"/>
+<label x="15.24" y="127" size="1.778" layer="95"/>
+<pinref part="R14" gate="G$1" pin="2"/>
+</segment>
+<segment>
+<pinref part="DB9" gate="G$1" pin="1"/>
+<wire x1="0" y1="81.28" x2="0" y2="88.9" width="0.1524" layer="91"/>
+<label x="-2.54" y="88.9" size="1.778" layer="95"/>
+</segment>
+</net>
+<net name="RX1" class="0">
+<segment>
+<pinref part="SV2" gate="1" pin="6"/>
+<wire x1="-25.4" y1="-2.54" x2="-25.4" y2="-7.62" width="0.1524" layer="91"/>
+<label x="-22.86" y="-5.08" size="1.778" layer="95"/>
+</segment>
+<segment>
+<pinref part="CAN_TRANSCIEVER1" gate="G$1" pin="RXD"/>
+<wire x1="-20.32" y1="119.38" x2="-20.32" y2="109.22" width="0.1524" layer="91"/>
+<wire x1="-20.32" y1="109.22" x2="-38.1" y2="109.22" width="0.1524" layer="91"/>
+<label x="-17.78" y="109.22" size="1.778" layer="95"/>
+</segment>
+</net>
+<net name="TX1" class="0">
+<segment>
+<pinref part="SV2" gate="1" pin="5"/>
+<wire x1="-27.94" y1="-2.54" x2="-27.94" y2="-7.62" width="0.1524" layer="91"/>
+<label x="-33.02" y="-5.08" size="1.778" layer="95"/>
+</segment>
+<segment>
+<pinref part="CAN_TRANSCIEVER1" gate="G$1" pin="TXD"/>
+<wire x1="-20.32" y1="142.24" x2="-33.02" y2="142.24" width="0.1524" layer="91"/>
+<label x="-25.4" y="142.24" size="1.778" layer="95"/>
+</segment>
+</net>
