File: PCB/v2.0/MDAS_Controller_V2.sch (KiCad schematic (older format))
At the start: 95 parts, among them J1 JTAG, J2 DB9_Male, J3 DB15_Male, Q1 DTC114E, Q2 DTC114E, Q3 DTC114E, SW1 SW_DIP_x04, T2 TestPoint, T5 TestPoint, U1 TM4C123GH6PM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

Commit message: Redesign routing
Parts:
- added C26, C27: 0.01uF, Capacitor_SMD:C_0603_1608Metric_Pad1.05x0.95mm_HandSolder, symbol Device:C
- added R19, R20, R21, R22: 1k, Resistor_SMD:R_0603_1608Metric_Pad1.05x0.95mm_HandSolder, symbol Device:R_US
- renumbered GPI1 to SW1P1, GPI2 to SW2P1
Connections:
- net labels added: SW1P, SW2P
- net labels removed: GPI1P, GPI2P
- wire segments 335 -> 356
- no-connect marks 29 -> 32
Changed lines of the file:
@@
 Text GLabel 7150 3000 2    50   BiDi ~ 0
 SDA
-Text GLabel 7150 5100 2    50   Input ~ 0
-SW1
-Text GLabel 7150 5200 2    50   Input ~ 0
-SW2
+Text GLabel 7950 5000 2    50   Input ~ 0
+GPI1
+Text GLabel 7950 5250 2    50   Input ~ 0
+GPI2
 Text GLabel 4350 2500 0    50   Input ~ 0
-GPI1P
+SW1P
 Text GLabel 4350 2900 0    50   Input ~ 0
-GPI2P
+SW2P
 $Comp
 L power:GND #PWR08
@@
 Connection ~ 9750 4200
 Wire Wire Line
-	9750 4500 10650 4500
+	9750 4500 10000 4500
 Connection ~ 9750 4500
 Text GLabel 7150 2700 2    50   Input ~ 0
@@
 TXD
 Text GLabel 10550 8550 0    50   Input ~ 0
-GPI1
+SW1
 Text GLabel 10550 8650 0    50   Input ~ 0
-GPI2
+SW2
 Text GLabel 10550 8750 0    50   Input ~ 0
 T2
@@
 T5
 Text GLabel 10550 8950 0    50   Input ~ 0
-SW1
+GPI1
 Text GLabel 10550 9050 0    50   Input ~ 0
-SW2
+GPI2
 Text GLabel 10550 9150 0    50   Input ~ 0
 AI1H
@@
 $EndComp
 Text GLabel 8700 6700 0    50   Input ~ 0
-GPI1
+SW1
 $Comp
 L SamacSys_Parts:TPS70933DBVT U10
@@
 	1    0    0    -1
 $EndComp
-Text GLabel 10100 6800 2    50   Output ~ 0
-GPI1P
+Text GLabel 10400 6800 2    50   Output ~ 0
+SW1P
 Text GLabel 8700 7350 0    50   Input ~ 0
-GPI2
+SW2
 $Comp
 L SamacSys_Parts:TPS70933DBVT U11
@@
 	1    0    0    -1
 $EndComp
-Text GLabel 10100 7450 2    50   Output ~ 0
-GPI2P
+Text GLabel 10400 7450 2    50   Output ~ 0
+SW2P
 $Comp
 L Connector:TestPoint CAN1H1
@@
 $EndComp
 Wire Wire Line
-	9850 7450 10000 7450
-Wire Wire Line
-	10100 6800 10000 6800
-$Comp
-L Connector:TestPoint GPI1
+	10150 7450 10300 7450
+Wire Wire Line
+	10400 6800 10300 6800
+$Comp
+L Connector:TestPoint SW1P1
 U 1 1 5C37C0A0
-P 10000 6600
-F 0 "GPI1" H 10058 6720 50  0000 L CNN
-F 1 "TestPoint" H 10058 6629 50  0000 L CNN
-F 2 "TestPoint:TestPoint_Loop_D1.80mm_Drill1.0mm_Beaded" H 10200 6600 50  0001 C CNN
-F 3 "~" H 10200 6600 50  0001 C CNN
-	1    10000 6600
-	1    0    0    -1
-$EndComp
-$Comp
-L Connector:TestPoint GPI2
+P 10300 6600
+F 0 "SW1P1" H 10358 6720 50  0000 L CNN
+F 1 "TestPoint" H 10358 6629 50  0000 L CNN
+F 2 "TestPoint:TestPoint_Loop_D1.80mm_Drill1.0mm_Beaded" H 10500 6600 50  0001 C CNN
+F 3 "~" H 10500 6600 50  0001 C CNN
+	1    10300 6600
+	1    0    0    -1
+$EndComp
+$Comp
+L Connector:TestPoint SW2P1
 U 1 1 5C37C172
-P 10000 7300
-F 0 "GPI2" H 10058 7420 50  0000 L CNN
-F 1 "TestPoint" H 10058 7329 50  0000 L CNN
-F 2 "TestPoint:TestPoint_Loop_D1.80mm_Drill1.0mm_Beaded" H 10200 7300 50  0001 C CNN
-F 3 "~" H 10200 7300 50  0001 C CNN
-	1    10000 7300
-	1    0    0    -1
-$EndComp
-Wire Wire Line
-	10000 6600 10000 6800
-Connection ~ 10000 6800
-Wire Wire Line
-	10000 6800 9850 6800
-Wire Wire Line
-	10000 7300 10000 7450
-Connection ~ 10000 7450
-Wire Wire Line
-	10000 7450 10100 7450
+P 10300 7300
+F 0 "SW2P1" H 10358 7420 50  0000 L CNN
+F 1 "TestPoint" H 10358 7329 50  0000 L CNN
+F 2 "TestPoint:TestPoint_Loop_D1.80mm_Drill1.0mm_Beaded" H 10500 7300 50  0001 C CNN
+F 3 "~" H 10500 7300 50  0001 C CNN
+	1    10300 7300
+	1    0    0    -1
+$EndComp
+Wire Wire Line
+	10300 6600 10300 6800
+Connection ~ 10300 6800
+Wire Wire Line
+	10300 6800 10150 6800
+Wire Wire Line
+	10300 7300 10300 7450
+Connection ~ 10300 7450
+Wire Wire Line
+	10300 7450 10400 7450
 $Comp
 L Device:Jumper_NC_Small JP1
@@
 NoConn ~ 10650 4100
 NoConn ~ 10650 4300
-NoConn ~ 10650 4800
 NoConn ~ 4350 1800
 NoConn ~ 4350 2100
@@
 Wire Wire Line
 	1700 1650 2200 1650
+$Comp
+L Device:R_US R19
+U 1 1 5BA1CD78
+P 7750 5000
+F 0 "R19" V 7545 5000 50  0000 C CNN
+F 1 "1k" V 7636 5000 50  0000 C CNN
+F 2 "Resistor_SMD:R_0603_1608Metric_Pad1.05x0.95mm_HandSolder" V 7790 4990 50  0001 C CNN
+F 3 "~" H 7750 5000 50  0001 C CNN
+	1    7750 5000
+	0    1    1    0
+$EndComp
+$Comp
+L Device:R_US R20
+U 1 1 5BA1D4EF
+P 7750 5250
+F 0 "R20" V 7545 5250 50  0000 C CNN
+F 1 "1k" V 7636 5250 50  0000 C CNN
+F 2 "Resistor_SMD:R_0603_1608Metric_Pad1.05x0.95mm_HandSolder" V 7790 5240 50  0001 C CNN
+F 3 "~" H 7750 5250 50  0001 C CNN
+	1    7750 5250
+	0    1    1    0
+$EndComp
+$Comp
+L Device:C C26
+U 1 1 5BA1D5EA
+P 7200 5700
+F 0 "C26" H 7315 5746 50  0000 L CNN
+F 1 "0.01uF" H 7315 5655 50  0000 L CNN
+F 2 "Capacitor_SMD:C_0603_1608Metric_Pad1.05x0.95mm_HandSolder" H 7238 5550 50  0001 C CNN
+F 3 "~" H 7200 5700 50  0001 C CNN
+	1    7200 5700
+	1    0    0    -1
+$EndComp
+$Comp
+L Device:C C27
+U 1 1 5BA1D6E0
+P 7500 5700
+F 0 "C27" H 7615 5746 50  0000 L CNN
+F 1 "0.01uF" H 7615 5655 50  0000 L CNN
+F 2 "Capacitor_SMD:C_0603_1608Metric_Pad1.05x0.95mm_HandSolder" H 7538 5550 50  0001 C CNN
+F 3 "~" H 7500 5700 50  0001 C CNN
+	1    7500 5700
+	1    0    0    -1
+$EndComp
+Wire Wire Line
+	7250 5000 7250 5100
+Wire Wire Line
+	7250 5100 7150 5100
+Wire Wire Line
+	7950 5250 7900 5250
+Wire Wire Line
+	7950 5000 7900 5000
+Wire Wire Line
+	7250 5000 7350 5000
+Wire Wire Line
+	7600 5250 7500 5250
+Wire Wire Line
+	7250 5250 7250 5200
+Wire Wire Line
+	7250 5200 7150 5200
+Wire Wire Line
+	7200 5550 7200 5350
+Wire Wire Line
+	7200 5350 7350 5350
+Wire Wire Line
+	7350 5350 7350 5000
+Connection ~ 7350 5000
+Wire Wire Line
+	7350 5000 7600 5000
+Wire Wire Line
+	7500 5550 7500 5250
+Connection ~ 7500 5250
+Wire Wire Line
+	7500 5250 7250 5250
+Wire Wire Line
+	7500 5850 7500 5950
+Wire Wire Line
+	7500 5950 7350 5950
+Wire Wire Line
+	7200 5950 7200 5850
+$Comp
+L power:GND #PWR044
+U 1 1 5BBAF4A5
+P 7350 5950
+F 0 "#PWR044" H 7350 5700 50  0001 C CNN
+F 1 "GND" H 7355 5777 50  0000 C CNN
+F 2 "" H 7350 5950 50  0001 C CNN
+F 3 "" H 7350 5950 50  0001 C CNN
+	1    7350 5950
+	1    0    0    -1
+$EndComp
+Connection ~ 7350 5950
+Wire Wire Line
+	7350 5950 7200 5950
+$Comp
+L Device:R_US R21
+U 1 1 5BAF8D33
+P 10000 6800
+F 0 "R21" V 9795 6800 50  0000 C CNN
+F 1 "1k" V 9886 6800 50  0000 C CNN
+F 2 "Resistor_SMD:R_0603_1608Metric_Pad1.05x0.95mm_HandSolder" V 10040 6790 50  0001 C CNN
+F 3 "~" H 10000 6800 50  0001 C CNN
+	1    10000 6800
+	0    1    1    0
+$EndComp
+$Comp
+L Device:R_US R22
+U 1 1 5BAF9206
+P 10000 7450
+F 0 "R22" V 9795 7450 50  0000 C CNN
+F 1 "1k" V 9886 7450 50  0000 C CNN
+F 2 "Resistor_SMD:R_0603_1608Metric_Pad1.05x0.95mm_HandSolder" V 10040 7440 50  0001 C CNN
+F 3 "~" H 10000 7450 50  0001 C CNN
+	1    10000 7450
+	0    1    1    0
+$EndComp
+Wire Wire Line
+	10650 4800 10000 4800
+Wire Wire Line
+	10000 4800 10000 4500
+Connection ~ 10000 4500
+Wire Wire Line
+	10000 4500 10650 4500
+NoConn ~ 1000 4100
+NoConn ~ 1300 4100
+NoConn ~ 1300 4400
+NoConn ~ 1000 4400
 $EndSCHEMATC
